File: AMP_UN7+T.brd (EAGLE design)
At the start: 11 parts

Commit message: .
Parts:
- added 1C10: 1000m, rcl:E7,5-16
- added 1C4*: 330, rcl:C050-030X075
- added 1C5: 470, rcl:C050-030X075
- added 1C6: 100n, rcl:C150-072X183
- added 1C7: 100m, rcl:E2,5-7
- added 1C8: 10m, rcl:E2,5-7
- added 1C9: 2000m, rcl:E7,5-16
- added 1R10*: 1k, rcl:R0805
- added 1R3: 47k, rcl:RTRIM3296W
- added 1R8: 100 0.5w, rcl:0207/15
- added 1R9: 1 0.5w, rcl:0207/15
- added U$1: (no value), k174un7:25X25
- moved 1R7 153.9 mm to (-147.3, 86.4)
- moved 1R4 153.4 mm to (-139.7, 85.1)
- moved 1C3 153.4 mm to (-124.5, 61.0), turned to 90 degrees
- moved 1R1 151.0 mm to (-130.8, 83.8)
- moved 1C1 139.5 mm to (-124.5, 76.2), turned to 270 degrees
- moved DA1 139.5 mm to (-133.3, 44.5)
- moved 1C2 139.0 mm to (-110.5, 78.7)
- moved 1R5 127.2 mm to (-104.1, 87.6)
- moved 1R6 126.7 mm to (-120.7, 66.0)
- moved VT1 124.8 mm to (-106.7, 55.9)
- moved 1R2 115.4 mm to (-94.0, 74.9)
Connections:
- removed net 4++U: DA1.4
- new net +12V: 1C10.+, 1R7.2, 1R8.2, DA1.1
- new net N$11: 1C4*.1, 1C5.2, DA1.5
- new net N$12: 1C6.2, 1R9.2
- new net N$13: 1C8.-, 1R10*.1, DA1.6
- new net N$9: 1C7.+, 1R8.1, DA1.4
- new net OUT1+: 1C5.1, 1C6.1, 1C7.-, DA1.12
- new net OUT1-: 1C9.+, 1R10*.2
- net GND: now also 1C10.-, 1C4*.2, 1C9.-, 1R3.2, 1R3.3, 1R9.1
- net N$3: now also 1R3.1
- net N$5: now also 1C8.+
- net N$7: now also 1C1.+; no longer 1R7.2, DA1.1
Routing:
- net GND: track 0.00 -> 69.3 mm

Commit message: .
Parts:
- added 12V, IN, OUT: (no value), pinhead:1X02
- added HEATSINK1: (no value), k174un7:H_VELS
- added U$2: (no value), untitled:40X40
- 1C9: value 2000m -> 2000m(10000m)
- 1R8: device rcl:0207/15 -> rcl:0207/2V
- U$1: device k174un7:25X25 -> untitled:40X40
- moved 1R7 64.3 mm to (-108.0, 35.6)
- moved 1R4 49.4 mm to (-104.1, 50.8), turned to 180 degrees
- moved 1R5 38.4 mm to (-109.2, 49.5), turned to 180 degrees
- moved 1R10* 38.2 mm to (-129.5, 44.5), turned to 0 degrees
- moved 1R1 36.6 mm to (-110.5, 53.3), turned to 0 degrees
- moved 1C1 36.1 mm to (-96.5, 53.3), turned to 180 degrees
- moved 1R2 31.8 mm to (-113.0, 49.5)
- moved U$1 25.2 mm to (-152.4, 27.9)
- moved 1C2 18.2 mm to (-106.7, 61.0), turned to 180 degrees
- moved VT1 12.5 mm to (-118.1, 50.8)
- moved 1R6 11.5 mm to (-121.9, 54.6), turned to 270 degrees
- moved 1C8 8.03 mm to (-109.2, 44.5)
- moved 1C9 8.03 mm to (-142.2, 67.3), turned to 0 degrees
- moved 1C7 6.48 mm to (-149.9, 39.4)
- moved 1C10 5.68 mm to (-111.8, 21.6), turned to 180 degrees
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Connections:
- net +12V: now also 12V.2
- net GND: now also 12V.1, IN.2
- net N$7: now also IN.1
- net OUT1+: now also OUT.1
- net OUT1-: now also OUT.2
Routing:
- net N$11: track 0.00 -> 35.5 mm
- net N$9: track 0.00 -> 32.8 mm
- net OUT1+: track 0.00 -> 25.2 mm
- net GND: track 69.3 -> 93.3 mm
- net N$3: track 0.00 -> 15.8 mm
- net OUT1-: track 0.00 -> 13.8 mm
- net N$8: track 0.00 -> 13.7 mm
- net +12V: track 0.00 -> 11.9 mm
- net N$13: track 0.00 -> 7.94 mm

Commit message: .
Parts:
- 1C1, 1C2, 1C7, 1C8: device rcl:E2,5-7 -> rcl:E2,5-5
- 1C10, 1C9: device rcl:E7,5-16 -> rcl:E5-13
- 1C3: device rcl:E2,5-7 -> rcl:E2,5-6
- 1C6: device rcl:C150-072X183 -> rcl:C102-064X133
- moved U$2 139.6 mm to (17.8, 78.7), turned to 90 degrees
- moved U$1 139.1 mm to (-22.9, 78.7), turned to 90 degrees
- moved 1R8 133.7 mm to (-25.4, 82.5), turned to 90 degrees
- moved 1C10 130.2 mm to (-21.6, 115.6), turned to 270 degrees
- moved 1C7 122.9 mm to (-34.3, 81.3), turned to 180 degrees
- moved 12V 118.9 mm to (-31.8, 139.7), turned to 270 degrees
- moved 1R7 117.0 mm to (-30.5, 123.2), turned to 270 degrees
- moved 1C5 108.4 mm to (-44.5, 82.5), turned to 0 degrees
- moved DA1 108.1 mm to (-39.4, 97.8), turned to 90 degrees
- moved HEATSINK1 108.1 mm to (-39.4, 97.8), turned to 90 degrees
- moved 1R10* 107.4 mm to (-39.4, 102.9), turned to 270 degrees
- moved 1C4* 106.2 mm to (-38.1, 113.0), turned to 180 degrees
- moved 1C8 104.3 mm to (-39.4, 121.9), turned to 270 degrees
- moved OUT 98.3 mm to (-53.3, 82.5), turned to 90 degrees
- moved 1C6 97.9 mm to (-58.4, 61.0), turned to 180 degrees
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Routing:
- net GND: track 93.3 -> 87.1 mm
- net OUT1-: track 13.8 -> 11.3 mm
- net N$3: track 15.8 -> 17.4 mm
- net N$13: track 7.94 -> 6.67 mm
- net N$8: track 13.7 -> 13.0 mm
- net N$11: track 35.5 -> 36.0 mm

Commit message: .
Parts:
- removed 12V: (no value), pinhead:1X02
- added +12V: CON_2P, DSS:CON_PWR_2PIN4MM
- added 1C11, 1C4: 2000m(10000m), rcl:E5-13
- added HEATSINK2: (no value), k174un7:H_VELS
- moved 1C6 35.7 mm to (-61.0, 96.5), turned to 90 degrees
- moved 1R5 12.0 mm to (-36.8, 114.3)
- moved 1R4 11.7 mm to (-38.1, 118.1)
- moved 1C1 10.5 mm to (-50.8, 124.5), turned to 0 degrees
- moved 1C8 9.16 mm to (-31.8, 116.8)
- moved 1R2 8.98 mm to (-41.9, 116.8), turned to 180 degrees
- moved 1R1 6.48 mm to (-45.7, 119.4)
- moved 1C4* 6.48 mm to (-31.8, 111.8)
- moved OUT 5.24 mm to (-48.3, 81.3), turned to 180 degrees
- moved 1C10 4.58 mm to (-19.1, 111.8), turned to 180 degrees
- moved 1R8 4.02 mm to (-29.2, 81.3), turned to 0 degrees
- moved 1R6 4.02 mm to (-47.0, 109.2)
- moved 1C9 3.59 mm to (-55.9, 86.4)
- moved IN 3.59 mm to (-59.7, 121.9)
- moved VT1 2.84 mm to (-43.2, 111.8), turned to 180 degrees
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Connections:
- net +12V: now also +12V.2; no longer 12V.2
- net GND: now also +12V.1; no longer 12V.1
Routing:
- net +12V: track 11.9 -> 81.8 mm
- net GND: track 87.1 -> 138.4 mm
- net N$6: track 0.00 -> 27.5 mm
- net N$13: track 6.67 -> 17.1 mm
- net N$5: track 0.00 -> 8.12 mm
- net N$1: track 0.00 -> 7.65 mm
- net N$9: track 32.8 -> 25.7 mm
- net N$4: track 0.00 -> 5.62 mm
- net OUT1+: track 25.5 -> 20.0 mm
- net N$11: track 36.0 -> 34.1 mm
- net N$3: track 17.4 -> 19.0 mm
- net OUT1-: track 11.3 -> 12.5 mm

Commit message: 1
Parts:
- added 1R8': (no value), rcl:R1210W
- 1C4*: device rcl:C050-030X075 -> rcl:C050-025X075
- 1C6: device rcl:C102-064X133 -> rcl:C075-052X106
- 1R10*: device rcl:R0805 -> rcl:0207/12
- 1R8: device rcl:0207/2V -> rcl:R1210W
- 1R9: device rcl:0207/15 -> rcl:0411V
- moved U$1 40.4 mm to (-62.9, 84.5), turned to 0 degrees
- moved U$2 40.4 mm to (-22.2, 84.5), turned to 0 degrees
- moved 1C4 32.0 mm to (1.91, 62.2)
- moved 1C9 30.5 mm to (-55.2, 116.8), turned to 0 degrees
- moved 1C7 30.3 mm to (-24.1, 109.9), turned to 270 degrees
- moved IN 21.3 mm to (-38.4, 121.6), turned to 0 degrees
- moved 1C5 15.4 mm to (-40.0, 97.8), turned to 90 degrees
- moved 1R10* 15.0 mm to (-40.3, 117.8), flipped to the top, turned to 180 degrees
- moved 1R2 14.0 mm to (-50.8, 106.0), turned to 270 degrees
- moved VT1 13.9 mm to (-55.9, 106.0), turned to 90 degrees
- moved OUT 12.8 mm to (-59.7, 87.0)
- moved 1C2 11.3 mm to (-45.1, 113.7), turned to 180 degrees
- moved +12V 10.8 mm to (-19.7, 89.5)
- moved 1C10 10.8 mm to (-19.7, 101.0)
- moved 1R7 10.4 mm to (-38.4, 117.2)
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Connections:
- new net N$10: 1R8'.2, 1R8.1
- net GND: now also 1R9.2; no longer 1R9.1
- net N$12: now also 1R9.1; no longer 1R9.2
- net N$9: now also 1R8'.1; no longer 1R8.1
Routing:
- net OUT1-: track 12.5 -> 46.6 mm
- net OUT1+: track 20.0 -> 51.2 mm
- net N$6: track 27.5 -> 7.20 mm
- net N$1: track 7.65 -> 24.0 mm
- net N$11: track 34.1 -> 18.3 mm
- net GND: track 138.4 -> 127.9 mm, vias 0 -> 1
- net N$9: track 25.7 -> 18.2 mm
- net N$4: track 5.62 -> 11.9 mm
- net N$10: track 0.00 -> 6.04 mm
- net N$13: track 17.1 -> 11.8 mm
- net N$12: track 0.00 -> 4.90 mm
- net N$8: track 13.0 -> 17.4 mm
- net N$3: track 19.0 -> 15.4 mm
- net N$7: track 0.00 -> 3.51 mm
- net N$2: track 0.00 -> 2.86 mm
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
Commit message: 2
Parts:
- removed 1C11, 1C4: 2000m(10000m), rcl:E5-13
- added 1C12, C11: 100n, rcl:C0805
- moved +12V 0.95 mm to (-20.6, 89.5)
- moved U$2 0.63 mm to (-22.9, 84.5)
- moved 1C10 0.32 mm to (-19.4, 101.0), turned to 0 degrees
Connections:
- net +12V: now also +12V.1, C11.1; no longer +12V.2
- net GND: now also +12V.2, 1C12.2, C11.2; no longer +12V.1
- net N$6: now also 1C12.1
Routing:
- net +12V: track 84.5 -> 61.4 mm
- net GND: track 127.9 -> 137.7 mm, vias 1 -> 2
- net N$15: track 0.00 -> 2.54 mm
- net N$14: track 0.00 -> 2.54 mm
- net N$6: track 7.20 -> 9.55 mm

Commit message: .
Parts:
- moved 1C7 4.27 mm to (-27.0, 113.0), turned to 0 degrees
- moved 1C4* 3.72 mm to (-31.1, 116.5), turned to 90 degrees
- moved C11 1.14 mm to (-20.6, 94.6)
Routing:
- net GND: track 137.7 -> 147.7 mm, vias 2 -> 3
- net OUT1+: track 51.0 -> 54.5 mm
- net +12V: track 61.4 -> 63.6 mm
- net N$11: track 18.3 -> 19.8 mm
- net N$9: track 18.2 -> 17.0 mm
Changed lines of the file:
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@@
 <attribute name="VALUE" x="-27.94" y="93.98" size="1.27" layer="28" rot="MR270"/>
 </element>
-<element name="1C7" library="rcl" package="E2,5-5" value="100m" x="-24.13" y="109.855" smashed="yes" rot="R270">
-<attribute name="NAME" x="-25.8445" y="113.03" size="1.27" layer="25" ratio="10"/>
-<attribute name="VALUE" x="-26.543" y="107.442" size="1.27" layer="27" ratio="10" rot="R270"/>
-</element>
-<element name="1C4*" library="rcl" package="C050-025X075" value="330" x="-29.845" y="113.03" smashed="yes">
-<attribute name="NAME" x="-29.7815" y="114.681" size="1.27" layer="25" ratio="10"/>
-<attribute name="VALUE" x="-33.274" y="110.236" size="1.27" layer="27" ratio="10"/>
+<element name="1C7" library="rcl" package="E2,5-5" value="100m" x="-26.9875" y="113.03" smashed="yes">
+<attribute name="NAME" x="-30.1625" y="111.3155" size="1.27" layer="25" ratio="10" rot="R90"/>
+<attribute name="VALUE" x="-24.5745" y="110.617" size="1.27" layer="27" ratio="10"/>
+</element>
+<element name="1C4*" library="rcl" package="C050-025X075" value="330" x="-31.115" y="116.5225" smashed="yes" rot="R90">
+<attribute name="NAME" x="-32.766" y="116.586" size="1.27" layer="25" ratio="10" rot="R90"/>
+<attribute name="VALUE" x="-28.321" y="113.0935" size="1.27" layer="27" ratio="10" rot="R90"/>
 </element>
 <element name="1C5" library="rcl" package="C050-030X075" value="470" x="-40.005" y="97.79" smashed="yes" rot="R90">
@@
 <attribute name="VALUE" x="-59.817" y="112.903" size="1.778" layer="27" ratio="10"/>
 </element>
-<element name="1C10" library="rcl" package="E5-13" value="1000m" x="-19.3675" y="100.965"/>
+<element name="1C10" library="rcl" package="E5-13" value="1000m" x="-19.3675" y="100.965" smashed="yes">
+<attribute name="NAME" x="-21.5646" y="103.4923" size="1.778" layer="25" ratio="10"/>
+<attribute name="VALUE" x="-23.9395" y="97.028" size="1.778" layer="27" ratio="10"/>
+</element>
 <element name="1R3" library="rcl" package="RTRIM3296W" value="47k" x="-59.69" y="105.41" smashed="yes" rot="R180">
 <attribute name="NAME" x="-57.5775" y="103.7675" size="1.27" layer="25" rot="R90"/>
@@
 <attribute name="VALUE" x="-32.385" y="100.965" size="1.27" layer="28" rot="MR270"/>
 </element>
-<element name="C11" library="rcl" package="C0805" value="100n" x="-19.685" y="95.25" rot="MR180"/>
+<element name="C11" library="rcl" package="C0805" value="100n" x="-20.6375" y="94.615" rot="MR180"/>
 <element name="1C12" library="rcl" package="C0805" value="100n" x="-45.085" y="111.4425" smashed="yes" rot="MR0">
 <attribute name="NAME" x="-46.99" y="109.855" size="1.27" layer="26" rot="MR180"/>
@@
 <wire x1="-61.595" y1="106.045" x2="-62.23" y2="109.855" width="0.4064" layer="1"/>
 <wire x1="-62.23" y1="109.855" x2="-52.705" y2="116.84" width="0.4064" layer="1"/>
-<wire x1="-27.305" y1="113.03" x2="-16.8275" y2="100.965" width="0.4064" layer="1"/>
-<wire x1="-16.8275" y1="100.965" x2="-27.94" y2="93.98" width="0.4064" layer="1"/>
 <wire x1="-27.94" y1="93.98" x2="-39.37" y2="97.155" width="0.4064" layer="1"/>
 <wire x1="-46.355" y1="113.665" x2="-52.705" y2="116.84" width="0.4064" layer="1"/>
@@
 <wire x1="-46.355" y1="113.665" x2="-46.355" y2="111.7625" width="0.6096" layer="16"/>
 <wire x1="-46.355" y1="111.7625" x2="-46.035" y2="111.4425" width="0.6096" layer="16"/>
-<wire x1="-18.6375" y1="89.535" x2="-17.685" y2="95.5675" width="1.27" layer="16"/>
-<wire x1="-17.685" y1="95.5675" x2="-17.685" y2="100.1075" width="1.27" layer="16"/>
-<wire x1="-17.685" y1="100.1075" x2="-16.8275" y2="100.965" width="1.27" layer="16"/>
-<wire x1="-18.735" y1="95.25" x2="-18.0025" y2="95.25" width="0.6096" layer="16"/>
-<wire x1="-18.0025" y1="95.25" x2="-17.685" y2="95.5675" width="0.6096" layer="16"/>
-<via x="-56.1975" y="100.965" extent="1-16" drill="0.8" diameter="2.3"/>
+<via x="-55.88" y="100.965" extent="1-16" drill="0.8" diameter="2.3"/>
 <wire x1="-52.07" y1="100.6475" x2="-54.9275" y2="100.6475" width="0.6096" layer="1"/>
-<wire x1="-54.9275" y1="100.6475" x2="-56.1975" y2="100.965" width="0.6096" layer="1"/>
+<wire x1="-54.9275" y1="100.6475" x2="-55.88" y2="100.965" width="0.6096" layer="1"/>
 <wire x1="-59.69" y1="98.425" x2="-59.69" y2="100.965" width="0.6096" layer="16"/>
 <wire x1="-59.69" y1="100.965" x2="-59.69" y2="102.87" width="0.6096" layer="16"/>
-<wire x1="-56.1975" y1="100.965" x2="-59.69" y2="100.965" width="0.6096" layer="16"/>
+<wire x1="-55.88" y1="100.965" x2="-59.69" y2="100.965" width="0.6096" layer="16"/>
+<wire x1="-18.6375" y1="89.535" x2="-18.6375" y2="94.615" width="1.27" layer="16"/>
+<wire x1="-18.6375" y1="94.615" x2="-18.6375" y2="97.5675" width="1.27" layer="16"/>
+<wire x1="-19.6875" y1="94.615" x2="-18.6375" y2="94.615" width="1.27" layer="16"/>
+<via x="-18.6375" y="97.5675" extent="1-16" drill="0.8" diameter="2.3"/>
+<wire x1="-18.6375" y1="97.5675" x2="-28.8925" y2="100.6475" width="0.6096" layer="1"/>
+<wire x1="-28.8925" y1="100.6475" x2="-31.115" y2="119.0625" width="0.6096" layer="1"/>
+<wire x1="-18.6375" y1="97.5675" x2="-27.94" y2="93.98" width="0.6096" layer="1"/>
+<wire x1="-18.6375" y1="97.5675" x2="-16.8275" y2="100.965" width="1.27" layer="16"/>
 </signal>
 <signal name="N$3">
@@
 <wire x1="-43.18" y1="106.68" x2="-44.45" y2="106.68" width="0.6096" layer="16"/>
 <wire x1="-44.45" y1="106.68" x2="-48.895" y2="102.235" width="0.6096" layer="16"/>
-<wire x1="-48.895" y1="102.235" x2="-51.435" y2="102.235" width="0.6096" layer="16"/>
-<wire x1="-51.435" y1="102.235" x2="-55.245" y2="98.425" width="0.6096" layer="16"/>
-<wire x1="-55.245" y1="98.425" x2="-57.15" y2="98.425" width="0.6096" layer="16"/>
+<wire x1="-48.895" y1="102.235" x2="-51.1175" y2="102.235" width="0.6096" layer="16"/>
+<wire x1="-51.1175" y1="102.235" x2="-54.9275" y2="98.425" width="0.6096" layer="16"/>
+<wire x1="-54.9275" y1="98.425" x2="-57.15" y2="98.425" width="0.6096" layer="16"/>
 </signal>
 <signal name="N$9">
@@
 <wire x1="-33.655" y1="101.6" x2="-29.21" y2="106.045" width="0.6096" layer="16"/>
 <wire x1="-29.21" y1="106.045" x2="-29.21" y2="107.95" width="0.6096" layer="16"/>
-<wire x1="-24.13" y1="111.125" x2="-26.035" y2="111.125" width="0.6096" layer="16"/>
-<wire x1="-26.035" y1="111.125" x2="-29.21" y2="107.95" width="0.6096" layer="16"/>
+<wire x1="-28.2575" y1="113.03" x2="-28.8925" y2="111.125" width="0.6096" layer="16"/>
+<wire x1="-28.8925" y1="111.125" x2="-29.21" y2="107.95" width="0.6096" layer="16"/>
 </signal>
 <signal name="OUT1+">
@@
 <wire x1="-31.4325" y1="101.6" x2="-30.1625" y2="101.6" width="0.6096" layer="16"/>
 <wire x1="-30.1625" y1="101.6" x2="-26.67" y2="105.0925" width="0.6096" layer="16"/>
-<wire x1="-24.13" y1="108.585" x2="-26.67" y2="106.045" width="0.6096" layer="16"/>
+<wire x1="-25.7175" y1="113.03" x2="-26.67" y2="106.045" width="0.6096" layer="16"/>
 <wire x1="-26.67" y1="106.045" x2="-26.67" y2="105.0925" width="0.6096" layer="16"/>
 <wire x1="-40.005" y1="95.25" x2="-40.005" y2="95.885" width="0.6096" layer="16"/>
@@
 <wire x1="-35.56" y1="104.14" x2="-33.9725" y2="104.14" width="0.6096" layer="16"/>
 <wire x1="-33.9725" y1="104.14" x2="-32.385" y2="105.7275" width="0.6096" layer="16"/>
-<wire x1="-32.385" y1="105.7275" x2="-32.385" y2="113.03" width="0.6096" layer="16"/>
+<wire x1="-32.385" y1="105.7275" x2="-32.385" y2="112.7125" width="0.6096" layer="16"/>
+<wire x1="-32.385" y1="112.7125" x2="-31.115" y2="113.9825" width="0.6096" layer="16"/>
 </signal>
 <signal name="N$12">
@@
 <wire x1="-32.156" y1="88.9" x2="-31.115" y2="89.941" width="0.6096" layer="16"/>
 <contactref element="C11" pad="1"/>
-<wire x1="-21.9075" y1="95.25" x2="-21.9075" y2="97.4725" width="1.27" layer="16"/>
-<wire x1="-21.9075" y1="97.4725" x2="-21.9075" y2="100.965" width="1.27" layer="16"/>
-<wire x1="-21.9075" y1="95.25" x2="-21.9075" y2="93.25" width="1.27" layer="16"/>
-<wire x1="-21.9075" y1="93.25" x2="-22.6375" y2="89.535" width="1.27" layer="16"/>
-<wire x1="-20.635" y1="95.25" x2="-21.9075" y2="95.25" width="0.6096" layer="16"/>
 <wire x1="-21.9075" y1="100.965" x2="-21.9075" y2="112.0775" width="0.6096" layer="16"/>
-<wire x1="-21.9075" y1="112.0775" x2="-26.3525" y2="116.5225" width="0.6096" layer="16"/>
-<wire x1="-26.3525" y1="116.5225" x2="-29.21" y2="116.5225" width="0.6096" layer="16"/>
-<wire x1="-29.21" y1="116.5225" x2="-33.02" y2="120.3325" width="0.6096" layer="16"/>
+<wire x1="-21.9075" y1="112.0775" x2="-25.0825" y2="121.285" width="0.6096" layer="16"/>
+<wire x1="-25.0825" y1="121.285" x2="-27.94" y2="121.285" width="0.6096" layer="16"/>
+<wire x1="-27.94" y1="121.285" x2="-33.02" y2="120.3325" width="0.6096" layer="16"/>
 <wire x1="-34.29" y1="120.3325" x2="-37.465" y2="117.1575" width="0.6096" layer="16"/>
 <wire x1="-37.465" y1="117.1575" x2="-37.4675" y2="117.1575" width="0.6096" layer="16"/>
 <wire x1="-31.115" y1="89.941" x2="-29.439" y2="89.941" width="1.27" layer="16"/>
-<wire x1="-29.439" y1="89.941" x2="-21.9075" y2="97.4725" width="1.27" layer="16"/>
+<wire x1="-22.6375" y1="89.535" x2="-22.6375" y2="94.615" width="1.27" layer="16"/>
+<wire x1="-22.6375" y1="94.615" x2="-22.6375" y2="96.7425" width="1.27" layer="16"/>
+<wire x1="-22.6375" y1="96.7425" x2="-22.6375" y2="100.235" width="1.27" layer="16"/>
+<wire x1="-22.6375" y1="100.235" x2="-21.9075" y2="100.965" width="1.27" layer="16"/>
+<wire x1="-21.5875" y1="94.615" x2="-22.6375" y2="94.615" width="1.27" layer="16"/>
+<wire x1="-29.439" y1="89.941" x2="-22.6375" y2="96.7425" width="1.27" layer="16"/>
 </signal>
 <signal name="OUT1-">
@@
 <contactref element="1C1" pad="+"/>
 <contactref element="IN" pad="1"/>
-<wire x1="-43.18" y1="121.285" x2="-39.6875" y2="121.6025" width="0.4064" layer="16"/>
+<wire x1="-43.18" y1="121.285" x2="-42.8625" y2="121.6025" width="1.27" layer="16"/>
+<wire x1="-42.8625" y1="121.6025" x2="-39.6875" y2="121.6025" width="1.27" layer="16"/>
 </signal>
 <signal name="N$10">

Commit message: 3
Parts:
- removed 1C12: 100n, rcl:C0805
- added 1C13: 100m, rcl:E2,5-6
- added 1C14: 100m, rcl:E2,5-5
- added 1C15: 470, rcl:C050-030X075
- added 1C16: 100n, rcl:C075-052X106
- added 1C17, 1C4, 2C2: 10m, rcl:E2,5-5
- added 1C18: 2000m(10000m), rcl:E5-13
- added 1C4*1: 330, rcl:C050-025X075
- added 1R10, 1R14: 10k, rcl:R0805
- added 1R10*1: 1k, rcl:0207/12
- added 1R11: 330, rcl:R0805
- added 1R12: 150k, rcl:R0805
- added 1R13: 15k, rcl:R0805
- added 1R15: 5k1, rcl:R0805
- added 1R16: 100 0.5w, rcl:R1210W
- added 1R17: 1 0.5w, rcl:0411V
- added 1R18: 47k, rcl:RTRIM3296W
- added 1R8'1: (no value), rcl:R1210W
- added 2C10: 100n, rcl:C0805
- added C10: 1000m, rcl:E5-13
- added DA2: К174УН7, k174un7:DIL16-12
- added IN1, OUT1: (no value), pinhead:1X02
- added U$3: (no value), untitled:40X40
- added VT2: КТ3102Е, m_transistor:TO92
- 1C10: value 1000m -> 100n; device rcl:E5-13 -> rcl:C0805
- moved U$2 72.8 mm to (-14.9, 156.8)
- moved +12V 31.0 mm to (-26.4, 120.0), turned to 180 degrees
- moved C11 28.5 mm to (-26.4, 122.6), turned to 0 degrees
- moved 1C10 27.8 mm to (-45.1, 111.4), flipped to the bottom
Connections:
- new net N$16: 1R10.1, 1R12.2, DA2.8, VT2.1
- new net N$17: 1R11.2, VT2.3
- new net N$18: 1R12.1, 1R13.2, 1R18.1, VT2.2
- new net N$19: 1C4.-, 1R13.1
- new net N$20: 1C17.+, 1R10.2, 1R14.1
- new net N$21: 1R14.2, 1R15.1, 2C10.1, 2C2.+
- new net N$22: 1C13.+, DA2.7
- new net N$23: 1C14.+, 1R8'1.1, DA2.4
- new net N$24: 1C15.2, 1C4*1.1, DA2.5
- new net N$25: 1C16.2, 1R17.1
- new net N$26: 1C17.-, 1R10*1.1, DA2.6
- new net N$27: 1C4.+, IN1.1
- new net N$28: 1R16.1, 1R8'1.2
- new net OUT2+: 1C14.-, 1C15.1, 1C16.1, DA2.12, OUT1.1
- new net OUT2-: 1C18.+, 1R10*1.2, OUT1.2
- net +12V: now also 1R15.2, 1R16.2, C10.+, DA2.1; no longer 1C10.+
- net GND: now also 1C10.2, 1C13.-, 1C18.-, 1C4*1.2, 1R11.1, 1R17.2, 1R18.2, 1R18.3, 2C10.2, 2C2.-, C10.-, DA2.10, DA2.9, IN1.2; no longer 1C10.-, 1C12.2
- net N$6: now also 1C10.1; no longer 1C12.1
Routing:
- net OUT2+: track 0.00 -> 34.9 mm
- net N$24: track 0.00 -> 19.8 mm
- net N$16: track 0.00 -> 19.5 mm
- net GND: track 147.7 -> 166.6 mm
- net +12V: track 63.6 -> 82.0 mm
- net N$23: track 0.00 -> 17.0 mm
- net OUT2-: track 0.00 -> 14.4 mm
- net N$19: track 0.00 -> 11.9 mm
- net N$26: track 0.00 -> 11.8 mm
- net N$22: track 0.00 -> 9.78 mm
- net N$21: track 0.00 -> 9.55 mm
- net N$18: track 0.00 -> 6.30 mm
- net N$28: track 0.00 -> 6.04 mm
- net N$20: track 0.00 -> 5.40 mm
- net N$27: track 0.00 -> 3.62 mm
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