File: AMP_UN7+T.brd (EAGLE design)
At the start: 79.1 x 39.1 mm, 54 parts

Commit message: .
Parts:
- added 1C5', 2C5': (no value), rcl:C0805
- moved 1C1 0.32 mm to (27.3, 48.9)
- moved 1R6 0.32 mm to (15.6, 40.3)
Connections:
- removed net N$11: 1C4*.1, 1C5.2, DA1.5
- removed net N$24: 2C4*.1, 2C5.2, DA2.5
- new net DA1P5: 1C4*.1, 1C5'.2, 1C5.2, DA1.5
- new net DA2P5: 2C4*.1, 2C5'.2, 2C5.2, DA2.5
- net OUT1+: now also 1C5'.1
- net OUT2+: now also 2C5'.1
Routing:
- net DA1P5: track 0.00 -> 19.5 mm
- net DA2P5: track 0.00 -> 19.1 mm
- net N$11: track 17.9 -> 0.00 mm
- net N$24: track 17.5 -> 0.00 mm
- net IN1: track 4.26 -> 2.80 mm
- net +12V: track 145.2 -> 146.0 mm
- net OUT2+: track 56.7 -> 57.6 mm

Commit message: .
Parts:
- IN1, IN2, OUT1, OUT2: device pinhead:1X02 -> Разъёмы штырьковые 2.54мм:1X02
Routing:
- net N$29: track 0.00 -> 3.18 mm
- net N$11: track 0.00 -> 3.18 mm
- net N$27: track 0.00 -> 3.18 mm
- net N$24: track 0.00 -> 3.17 mm
Changed lines of the file:
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@@
 <attribute name="VALUE" x="6.21" y="38.4725" size="1.27" layer="27" rot="R270"/>
 </element>
-<element name="IN1" library="pinhead" package="1X02" value="" x="32.385" y="49.8475" smashed="yes">
+<element name="IN1" library="Разъёмы штырьковые 2.54мм" package="1X02" value="" x="32.385" y="49.8475" smashed="yes">
 <attribute name="NAME" x="33.2613" y="46.5963" size="1.27" layer="25" ratio="10"/>
 <attribute name="VALUE" x="29.845" y="46.6725" size="1.27" layer="27"/>
 </element>
-<element name="OUT1" library="pinhead" package="1X02" value="" x="11.43" y="15.24" smashed="yes" rot="R180">
+<element name="OUT1" library="Разъёмы штырьковые 2.54мм" package="1X02" value="" x="11.43" y="15.24" smashed="yes" rot="R180">
 <attribute name="NAME" x="11.8237" y="19.1262" size="1.27" layer="25" ratio="10" rot="R180"/>
 <attribute name="VALUE" x="13.97" y="18.415" size="1.27" layer="27" rot="R180"/>
@@
 <attribute name="VALUE" x="45.58" y="38.4725" size="1.27" layer="27" rot="R270"/>
 </element>
-<element name="IN2" library="pinhead" package="1X02" value="" x="70.485" y="48.895" smashed="yes">
+<element name="IN2" library="Разъёмы штырьковые 2.54мм" package="1X02" value="" x="70.485" y="48.895" smashed="yes">
 <attribute name="NAME" x="73.2663" y="50.7238" size="1.27" layer="25" ratio="10"/>
 <attribute name="VALUE" x="67.945" y="45.72" size="1.27" layer="27"/>
 </element>
-<element name="OUT2" library="pinhead" package="1X02" value="" x="47.625" y="15.24" smashed="yes" rot="R180">
+<element name="OUT2" library="Разъёмы штырьковые 2.54мм" package="1X02" value="" x="47.625" y="15.24" smashed="yes" rot="R180">
 <attribute name="NAME" x="44.5262" y="15.3162" size="1.27" layer="25" ratio="10" rot="R180"/>
 <attribute name="VALUE" x="50.165" y="18.415" size="1.27" layer="27" rot="R180"/>
@@
 <wire x1="69.215" y1="28.575" x2="69.215" y2="26.985" width="0.6096" layer="16"/>
 </signal>
+<signal name="N$11">
+<wire x1="8.5725" y1="52.3875" x2="6.985" y2="52.3875" width="0.3048" layer="16"/>
+<wire x1="6.985" y1="52.3875" x2="6.985" y2="50.8" width="0.3048" layer="16"/>
+</signal>
+<signal name="N$24">
+<wire x1="8.5725" y1="13.335" x2="6.985" y2="13.335" width="0.3048" layer="16"/>
+<wire x1="6.985" y1="13.335" x2="6.985" y2="14.9225" width="0.3048" layer="16"/>
+</signal>
+<signal name="N$27">
+<wire x1="84.455" y1="13.335" x2="86.0425" y2="13.335" width="0.3048" layer="16"/>
+<wire x1="86.0425" y1="13.335" x2="86.0425" y2="14.9225" width="0.3048" layer="16"/>
+</signal>
+<signal name="N$29">
+<wire x1="86.0425" y1="50.8" x2="86.0425" y2="52.3875" width="0.3048" layer="16"/>
+<wire x1="86.0425" y1="52.3875" x2="84.455" y2="52.3875" width="0.3048" layer="16"/>
+</signal>
 </signals>
