File: AMP_UN7+T.sch (EAGLE design)
At the start: 11 parts

Commit message: .
Parts:
- added 1C10: 1000m, rcl:CPOL-EUE7.5-16
- added 1C4*: 330, rcl:C-EU050-030X075
- added 1C5: 470, rcl:C-EU050-030X075
- added 1C6: 100n, rcl:C-EU150-072X183
- added 1C7: 100m, rcl:CPOL-EUE2.5-7
- added 1C8: 10m, rcl:CPOL-EUE2.5-7
- added 1C9: 2000m, rcl:CPOL-EUE7.5-16
- added 1R10*: 1k, rcl:R-EU_R0805
- added 1R3: 47k, rcl:R-TRIMM3296W
- added 1R8: 100 0.5w, rcl:R-EU_0207/15
- added 1R9: 1 0.5w, rcl:R-EU_0207/15
Connections:
- new net +12V: 1C10.+, 1R7.2, 1R8.2, DA1.1+V
- new net N$11: 1C4*.1, 1C5.2, DA1.5KOR
- new net N$12: 1C6.2, 1R9.2
- new net N$13: 1C8.-, 1R10*.1, DA1.6FB
- new net N$9: 1C7.+, 1R8.1, DA1.4++U
- new net OUT1+: 1C5.1, 1C6.1, 1C7.-, DA1.12OUT
- new net OUT1-: 1C9.+, 1R10*.2
- net GND: now also 1C10.-, 1C4*.2, 1C9.-, 1R3.E, 1R3.S, 1R9.1
- net N$3: now also 1R3.A
- net N$5: now also 1C8.+
- net N$7: now also 1C1.+; no longer 1R7.2, DA1.1+V
Other:
- note added: "1"
- note added: "2"
- note added: "3"
- note added: "4"
- note added: "5"
- note added: "6"
- note added: "7"
- note added: "8"
- moved on the sheet: 1C1, 1C2, 1C3, 1R1, 1R2, 1R4, 1R5, 1R6, 1R7, VT1

Commit message: .
Parts:
- added 12V, IN, OUT: (no value), pinhead:PINHD-1X2
- added HEATSINK1: HEATSINK_V, k174un7:HEATSINK_V
- 1C9: value 2000m -> 2000m(10000m)
- 1R8: device rcl:R-EU_0207/15 -> rcl:R-EU_0207/2V
Connections:
- net +12V: now also 12V.2
- net GND: now also 12V.1, IN.2
- net N$7: now also IN.1
- net OUT1+: now also OUT.1
- net OUT1-: now also OUT.2
Changed lines of the file:
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@@
 <part name="1C3" library="rcl" deviceset="CPOL-EU" device="E2.5-7" value="100m"/>
 <part name="GND4" library="supply1" deviceset="GND" device=""/>
-<part name="1R8" library="rcl" deviceset="R-EU_" device="0207/15" value="100 0.5w"/>
+<part name="1R8" library="rcl" deviceset="R-EU_" device="0207/2V" value="100 0.5w"/>
 <part name="1C7" library="rcl" deviceset="CPOL-EU" device="E2.5-7" value="100m"/>
 <part name="1C4*" library="rcl" deviceset="C-EU" device="050-030X075" value="330"/>
@@
 <part name="1R10*" library="rcl" deviceset="R-EU_" device="R0805" value="1k"/>
 <part name="P+1" library="supply1" deviceset="+12V" device=""/>
-<part name="1C9" library="rcl" deviceset="CPOL-EU" device="E7.5-16" value="2000m"/>
+<part name="1C9" library="rcl" deviceset="CPOL-EU" device="E7.5-16" value="2000m(10000m)"/>
 <part name="GND7" library="supply1" deviceset="GND" device=""/>
 <part name="1C10" library="rcl" deviceset="CPOL-EU" device="E7.5-16" value="1000m"/>
@@
 <part name="GND17" library="supply1" deviceset="GND" device=""/>
 <part name="GND10" library="supply1" deviceset="GND" device=""/>
+<part name="IN" library="pinhead" deviceset="PINHD-1X2" device=""/>
+<part name="OUT" library="pinhead" deviceset="PINHD-1X2" device=""/>
+<part name="12V" library="pinhead" deviceset="PINHD-1X2" device=""/>
+<part name="HEATSINK1" library="k174un7" deviceset="HEATSINK" device="_V" value=""/>
 </parts>
 <sheets>
@@
 <instance part="GND17" gate="1" x="38.1" y="101.6"/>
 <instance part="GND10" gate="1" x="90.17" y="118.11"/>
+<instance part="IN" gate="G$1" x="12.7" y="124.46" rot="MR0"/>
+<instance part="OUT" gate="G$1" x="142.24" y="111.76"/>
+<instance part="12V" gate="G$1" x="139.7" y="172.72"/>
+<instance part="HEATSINK1" gate="G$1" x="86.36" y="91.44" smashed="yes">
+<attribute name="NAME" x="79.375" y="97.155" size="1.778" layer="95"/>
+<attribute name="VALUE" x="78.74" y="88.9" size="1.778" layer="96"/>
+</instance>
 </instances>
 <busses>
@@
 <pinref part="GND8" gate="1" pin="GND"/>
 <wire x1="114.3" y1="152.4" x2="114.3" y2="149.86" width="0.1524" layer="91"/>
+<pinref part="12V" gate="G$1" pin="1"/>
+<wire x1="137.16" y1="175.26" x2="106.68" y2="175.26" width="0.1524" layer="91"/>
+<wire x1="106.68" y1="175.26" x2="109.22" y2="149.86" width="0.1524" layer="91"/>
+<wire x1="109.22" y1="149.86" x2="114.3" y2="149.86" width="0.1524" layer="91"/>
 </segment>
 <segment>
@@
 <pinref part="GND17" gate="1" pin="GND"/>
 <wire x1="38.1" y1="104.14" x2="38.1" y2="119.38" width="0.1524" layer="91"/>
-<wire x1="38.1" y1="119.38" x2="27.94" y2="119.38" width="0.1524" layer="91"/>
+<wire x1="38.1" y1="119.38" x2="30.48" y2="119.38" width="0.1524" layer="91"/>
+<pinref part="IN" gate="G$1" pin="2"/>
+<wire x1="30.48" y1="119.38" x2="27.94" y2="119.38" width="0.1524" layer="91"/>
+<wire x1="15.24" y1="124.46" x2="30.48" y2="124.46" width="0.1524" layer="91"/>
+<wire x1="30.48" y1="124.46" x2="30.48" y2="119.38" width="0.1524" layer="91"/>
 </segment>
 <segment>
@@
 <junction x="104.14" y="132.08"/>
 <wire x1="104.14" y1="134.62" x2="104.14" y2="132.08" width="0.1524" layer="91"/>
-<wire x1="111.76" y1="132.08" x2="134.62" y2="132.08" width="0.1524" layer="91"/>
+<wire x1="111.76" y1="132.08" x2="127" y2="132.08" width="0.1524" layer="91"/>
 <junction x="111.76" y="132.08"/>
 <label x="127" y="132.08" size="1.778" layer="95"/>
+<pinref part="OUT" gate="G$1" pin="1"/>
+<wire x1="127" y1="132.08" x2="134.62" y2="132.08" width="0.1524" layer="91"/>
+<wire x1="139.7" y1="114.3" x2="127" y2="114.3" width="0.1524" layer="91"/>
+<wire x1="127" y1="114.3" x2="127" y2="132.08" width="0.1524" layer="91"/>
 </segment>
 </net>
@@
 <wire x1="114.3" y1="160.02" x2="114.3" y2="162.56" width="0.1524" layer="91"/>
 <junction x="114.3" y="162.56"/>
+<pinref part="12V" gate="G$1" pin="2"/>
+<wire x1="137.16" y1="172.72" x2="114.3" y2="172.72" width="0.1524" layer="91"/>
+<wire x1="114.3" y1="172.72" x2="114.3" y2="162.56" width="0.1524" layer="91"/>
 </segment>
 </net>
@@
 <pinref part="1R10*" gate="G$1" pin="2"/>
 <wire x1="109.22" y1="93.98" x2="106.68" y2="93.98" width="0.1524" layer="91"/>
-<wire x1="109.22" y1="93.98" x2="134.62" y2="93.98" width="0.1524" layer="91"/>
+<wire x1="109.22" y1="93.98" x2="127" y2="93.98" width="0.1524" layer="91"/>
 <junction x="109.22" y="93.98"/>
 <label x="124.46" y="93.98" size="1.778" layer="95"/>
+<pinref part="OUT" gate="G$1" pin="2"/>
+<wire x1="127" y1="93.98" x2="134.62" y2="93.98" width="0.1524" layer="91"/>
+<wire x1="139.7" y1="111.76" x2="127" y2="111.76" width="0.1524" layer="91"/>
+<wire x1="127" y1="111.76" x2="127" y2="93.98" width="0.1524" layer="91"/>
 </segment>
 </net>
@@
 <segment>
 <pinref part="1C1" gate="G$1" pin="+"/>
-<wire x1="33.02" y1="132.08" x2="27.94" y2="132.08" width="0.1524" layer="91"/>
-</segment>
-</net>
+<wire x1="33.02" y1="132.08" x2="30.48" y2="132.08" width="0.1524" layer="91"/>
+<pinref part="IN" gate="G$1" pin="1"/>
+<wire x1="30.48" y1="132.08" x2="27.94" y2="132.08" width="0.1524" layer="91"/>
+<wire x1="15.24" y1="127" x2="30.48" y2="127" width="0.1524" layer="91"/>
+<wire x1="30.48" y1="127" x2="30.48" y2="132.08" width="0.1524" layer="91"/>
+</segment>
+</net>

Commit message: .
Parts:
- 1C1, 1C2, 1C7, 1C8: device rcl:CPOL-EUE2.5-7 -> rcl:CPOL-EUE2.5-5
- 1C10, 1C9: device rcl:CPOL-EUE7.5-16 -> rcl:CPOL-EUE5-13
- 1C3: device rcl:CPOL-EUE2.5-7 -> rcl:CPOL-EUE2.5-6
- 1C6: device rcl:C-EU150-072X183 -> rcl:C-EU102-064X133
Changed lines of the file:
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@@
 <part name="1R2" library="rcl" deviceset="R-EU_" device="R0805" value="150k"/>
 <part name="1R1" library="rcl" deviceset="R-EU_" device="R0805" value="15k"/>
-<part name="1C1" library="rcl" deviceset="CPOL-EU" device="E2.5-7" value="10m"/>
+<part name="1C1" library="rcl" deviceset="CPOL-EU" device="E2.5-5" value="10m"/>
 <part name="1R4" library="rcl" deviceset="R-EU_" device="R0805" value="10k"/>
-<part name="1C2" library="rcl" deviceset="CPOL-EU" device="E2.5-7" value="10m"/>
+<part name="1C2" library="rcl" deviceset="CPOL-EU" device="E2.5-5" value="10m"/>
 <part name="GND2" library="supply1" deviceset="GND" device=""/>
 <part name="1R7" library="rcl" deviceset="R-EU_" device="R0805" value="5k1"/>
-<part name="1C3" library="rcl" deviceset="CPOL-EU" device="E2.5-7" value="100m"/>
+<part name="1C3" library="rcl" deviceset="CPOL-EU" device="E2.5-6" value="100m"/>
 <part name="GND4" library="supply1" deviceset="GND" device=""/>
 <part name="1R8" library="rcl" deviceset="R-EU_" device="0207/2V" value="100 0.5w"/>
-<part name="1C7" library="rcl" deviceset="CPOL-EU" device="E2.5-7" value="100m"/>
+<part name="1C7" library="rcl" deviceset="CPOL-EU" device="E2.5-5" value="100m"/>
 <part name="1C4*" library="rcl" deviceset="C-EU" device="050-030X075" value="330"/>
 <part name="GND3" library="supply1" deviceset="GND" device=""/>
 <part name="1C5" library="rcl" deviceset="C-EU" device="050-030X075" value="470"/>
-<part name="1C6" library="rcl" deviceset="C-EU" device="150-072X183" value="100n"/>
+<part name="1C6" library="rcl" deviceset="C-EU" device="102-064X133" value="100n"/>
 <part name="1R9" library="rcl" deviceset="R-EU_" device="0207/15" value="1 0.5w"/>
 <part name="GND5" library="supply1" deviceset="GND" device=""/>
-<part name="1C8" library="rcl" deviceset="CPOL-EU" device="E2.5-7" value="10m"/>
+<part name="1C8" library="rcl" deviceset="CPOL-EU" device="E2.5-5" value="10m"/>
 <part name="GND6" library="supply1" deviceset="GND" device=""/>
 <part name="1R10*" library="rcl" deviceset="R-EU_" device="R0805" value="1k"/>
 <part name="P+1" library="supply1" deviceset="+12V" device=""/>
-<part name="1C9" library="rcl" deviceset="CPOL-EU" device="E7.5-16" value="2000m(10000m)"/>
+<part name="1C9" library="rcl" deviceset="CPOL-EU" device="E5-13" value="2000m(10000m)"/>
 <part name="GND7" library="supply1" deviceset="GND" device=""/>
-<part name="1C10" library="rcl" deviceset="CPOL-EU" device="E7.5-16" value="1000m"/>
+<part name="1C10" library="rcl" deviceset="CPOL-EU" device="E5-13" value="1000m"/>
 <part name="GND8" library="supply1" deviceset="GND" device=""/>
 <part name="1R3" library="rcl" deviceset="R-TRIMM" device="3296W" value="47k"/>

Commit message: .
Parts:
- removed 12V: (no value), pinhead:PINHD-1X2
- added +12V: CON_2P, DSS:CON_2P
- added 1C11, 1C4: 2000m(10000m), rcl:CPOL-EUE5-13
- added HEATSINK2: HEATSINK_V, k174un7:HEATSINK_V
Connections:
- net +12V: now also +12V.2; no longer 12V.2
- net GND: now also +12V.1; no longer 12V.1
Other:
- moved on the sheet: 1C10

Commit message: 1
Parts:
- added 1R8': (no value), rcl:R-EU_R1210W
- 1C4*: device rcl:C-EU050-030X075 -> rcl:C-EU050-025X075
- 1C6: device rcl:C-EU102-064X133 -> rcl:C-EU075-052X106
- 1R10*: device rcl:R-EU_R0805 -> rcl:R-EU_0207/12
- 1R8: device rcl:R-EU_0207/2V -> rcl:R-EU_R1210W
- 1R9: device rcl:R-EU_0207/15 -> rcl:R-EU_0411/3V
Connections:
- new net N$10: 1R8'.2, 1R8.1
- net GND: now also 1R9.2; no longer 1R9.1
- net N$12: now also 1R9.1; no longer 1R9.2
- net N$9: now also 1R8'.1; no longer 1R8.1
Other:
- moved on the sheet: 1C2, 1R4, 1R7, 1R8, 1R9

Commit message: 2
Parts:
- removed 1C11, 1C4: 2000m(10000m), rcl:CPOL-EUE5-13
- added 1C12, C11: 100n, rcl:C-EUC0805
Connections:
- net +12V: now also +12V.1, C11.1; no longer +12V.2
- net GND: now also +12V.2, 1C12.2, C11.2; no longer +12V.1
- net N$6: now also 1C12.1
Other:
- moved on the sheet: +12V
Changed lines of the file:
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@@
 <part name="+12V" library="DSS" deviceset="CON_2P" device=""/>
 <part name="P+2" library="supply1" deviceset="+12V" device=""/>
-<part name="1C4" library="rcl" deviceset="CPOL-EU" device="E5-13" value="2000m(10000m)"/>
-<part name="1C11" library="rcl" deviceset="CPOL-EU" device="E5-13" value="2000m(10000m)"/>
 <part name="1R8'" library="rcl" deviceset="R-EU_" device="R1210W"/>
+<part name="C11" library="rcl" deviceset="C-EU" device="C0805" value="100n"/>
+<part name="1C12" library="rcl" deviceset="C-EU" device="C0805" value="100n"/>
+<part name="GND11" library="supply1" deviceset="GND" device=""/>
 </parts>
 <sheets>
@@
 <attribute name="VALUE" x="182.88" y="96.52" size="1.778" layer="96"/>
 </instance>
-<instance part="+12V" gate="G$1" x="17.78" y="38.1"/>
-<instance part="P+2" gate="1" x="40.64" y="38.1" rot="R270"/>
-<instance part="1C4" gate="G$1" x="205.74" y="91.44" rot="MR0"/>
-<instance part="1C11" gate="G$1" x="231.14" y="81.28" rot="MR0"/>
+<instance part="+12V" gate="G$1" x="17.78" y="35.56" rot="MR180"/>
+<instance part="P+2" gate="1" x="55.88" y="38.1" rot="R270"/>
 <instance part="1R8'" gate="G$1" x="96.52" y="152.4" smashed="yes" rot="R90">
 <attribute name="NAME" x="102.87" y="155.9814" size="1.778" layer="95" rot="R180"/>
 <attribute name="VALUE" x="107.95" y="153.162" size="1.778" layer="96" rot="R180"/>
 </instance>
+<instance part="C11" gate="G$1" x="48.26" y="30.48"/>
+<instance part="1C12" gate="G$1" x="50.8" y="165.1" rot="MR0"/>
+<instance part="GND11" gate="1" x="50.8" y="154.94"/>
 </instances>
 <busses>
@@
 <wire x1="35.56" y1="22.86" x2="35.56" y2="20.32" width="0.1524" layer="91"/>
 <wire x1="35.56" y1="22.86" x2="27.94" y2="22.86" width="0.1524" layer="91"/>
-<pinref part="+12V" gate="G$1" pin="1"/>
+<pinref part="+12V" gate="G$1" pin="2"/>
 <wire x1="25.4" y1="35.56" x2="27.94" y2="35.56" width="0.1524" layer="91"/>
 <wire x1="27.94" y1="22.86" x2="27.94" y2="35.56" width="0.1524" layer="91"/>
 <junction x="35.56" y="22.86"/>
+<wire x1="35.56" y1="22.86" x2="48.26" y2="22.86" width="0.1524" layer="91"/>
+<pinref part="C11" gate="G$1" pin="2"/>
+<wire x1="48.26" y1="22.86" x2="48.26" y2="25.4" width="0.1524" layer="91"/>
 </segment>
 <segment>
@@
 <wire x1="90.17" y1="121.92" x2="90.17" y2="120.65" width="0.1524" layer="91"/>
 <pinref part="GND10" gate="1" pin="GND"/>
+</segment>
+<segment>
+<pinref part="1C12" gate="G$1" pin="2"/>
+<pinref part="GND11" gate="1" pin="GND"/>
+<wire x1="50.8" y1="160.02" x2="50.8" y2="157.48" width="0.1524" layer="91"/>
 </segment>
 </net>
@@
 <wire x1="71.12" y1="172.72" x2="76.2" y2="172.72" width="0.1524" layer="91"/>
 <junction x="71.12" y="172.72"/>
+<pinref part="1C12" gate="G$1" pin="1"/>
+<wire x1="50.8" y1="167.64" x2="50.8" y2="172.72" width="0.1524" layer="91"/>
+<wire x1="50.8" y1="172.72" x2="63.5" y2="172.72" width="0.1524" layer="91"/>
+<junction x="63.5" y="172.72"/>
 </segment>
 </net>
@@
 <segment>
 <pinref part="P+2" gate="1" pin="+12V"/>
-<wire x1="38.1" y1="38.1" x2="35.56" y2="38.1" width="0.1524" layer="91"/>
+<wire x1="53.34" y1="38.1" x2="48.26" y2="38.1" width="0.1524" layer="91"/>
 <pinref part="1C10" gate="G$1" pin="+"/>
+<wire x1="48.26" y1="38.1" x2="35.56" y2="38.1" width="0.1524" layer="91"/>
 <wire x1="35.56" y1="38.1" x2="35.56" y2="33.02" width="0.1524" layer="91"/>
-<pinref part="+12V" gate="G$1" pin="2"/>
+<pinref part="+12V" gate="G$1" pin="1"/>
 <wire x1="25.4" y1="38.1" x2="35.56" y2="38.1" width="0.1524" layer="91"/>
 <junction x="35.56" y="38.1"/>
-</segment>
-</net>
+<pinref part="C11" gate="G$1" pin="1"/>
+<wire x1="48.26" y1="33.02" x2="48.26" y2="38.1" width="0.1524" layer="91"/>
+<junction x="48.26" y="38.1"/>
+</segment>
+</net>

Commit message: 3
Parts:
- removed 1C12: 100n, rcl:C-EUC0805
- added 1C13: 100m, rcl:CPOL-EUE2.5-6
- added 1C14: 100m, rcl:CPOL-EUE2.5-5
- added 1C15: 470, rcl:C-EU050-030X075
- added 1C16: 100n, rcl:C-EU075-052X106
- added 1C17, 1C4, 2C2: 10m, rcl:CPOL-EUE2.5-5
- added 1C18: 2000m(10000m), rcl:CPOL-EUE5-13
- added 1C4*1: 330, rcl:C-EU050-025X075
- added 1R10, 1R14: 10k, rcl:R-EU_R0805
- added 1R10*1: 1k, rcl:R-EU_0207/12
- added 1R11: 330, rcl:R-EU_R0805
- added 1R12: 150k, rcl:R-EU_R0805
- added 1R13: 15k, rcl:R-EU_R0805
- added 1R15: 5k1, rcl:R-EU_R0805
- added 1R16: 100 0.5w, rcl:R-EU_R1210W
- added 1R17: 1 0.5w, rcl:R-EU_0411/3V
- added 1R18: 47k, rcl:R-TRIMM3296W
- added 1R8'1: (no value), rcl:R-EU_R1210W
- added 2C10: 100n, rcl:C-EUC0805
- added C10: 1000m, rcl:CPOL-EUE5-13
- added DA2: К174УН7, k174un7:K174UN7
- added IN1, OUT1: (no value), pinhead:PINHD-1X2
- added VT2: КТ3102Е, m_transistor:BJT_NPN_TO-92_CBE
- 1C10: value 1000m -> 100n; device rcl:CPOL-EUE5-13 -> rcl:C-EUC0805
Connections:
- new net N$16: 1R10.1, 1R12.2, DA2.8IN, VT2.C
- new net N$17: 1R11.2, VT2.E
- new net N$18: 1R12.1, 1R13.2, 1R18.A, VT2.B
- new net N$19: 1C4.-, 1R13.1
- new net N$20: 1C17.+, 1R10.2, 1R14.1
- new net N$21: 1R14.2, 1R15.1, 2C10.1, 2C2.+
- new net N$22: 1C13.+, DA2.7FILTR
- new net N$23: 1C14.+, 1R8'1.1, DA2.4++U
- new net N$24: 1C15.2, 1C4*1.1, DA2.5KOR
- new net N$25: 1C16.2, 1R17.1
- new net N$26: 1C17.-, 1R10*1.1, DA2.6FB
- new net N$27: 1C4.+, IN1.1
- new net N$28: 1R16.1, 1R8'1.2
- new net OUT2+: 1C14.-, 1C15.1, 1C16.1, DA2.12OUT, OUT1.1
- new net OUT2-: 1C18.+, 1R10*1.2, OUT1.2
- net +12V: now also 1R15.2, 1R16.2, C10.+, DA2.1+V; no longer 1C10.+
- net GND: now also 1C10.2, 1C13.-, 1C18.-, 1C4*1.2, 1R11.1, 1R17.2, 1R18.E, 1R18.S, 2C10.2, 2C2.-, C10.-, DA2.10E, DA2.9-V, IN1.2; no longer 1C10.-, 1C12.2
- net N$6: now also 1C10.1; no longer 1C12.1
Other:
- moved on the sheet: HEATSINK2

Commit message: 4
Parts:
- removed 1C13: 100m, rcl:CPOL-EUE2.5-6
- removed 1C14: 100m, rcl:CPOL-EUE2.5-5
- removed 1C15: 470, rcl:C-EU050-030X075
- removed 1C16: 100n, rcl:C-EU075-052X106
- removed 1C17, 1C4: 10m, rcl:CPOL-EUE2.5-5
- removed 1C18: 2000m(10000m), rcl:CPOL-EUE5-13
- removed 1C4*1: 330, rcl:C-EU050-025X075
- removed 1R10, 1R14: 10k, rcl:R-EU_R0805
- removed 1R10*1: 1k, rcl:R-EU_0207/12
- removed 1R11: 330, rcl:R-EU_R0805
- removed 1R12: 150k, rcl:R-EU_R0805
- removed 1R13: 15k, rcl:R-EU_R0805
- removed 1R15: 5k1, rcl:R-EU_R0805
- removed 1R16: 100 0.5w, rcl:R-EU_R1210W
- removed 1R17: 1 0.5w, rcl:R-EU_0411/3V
- removed 1R18: 47k, rcl:R-TRIMM3296W
- removed 1R8'1: (no value), rcl:R-EU_R1210W
- removed C10: 1000m, rcl:CPOL-EUE5-13
- removed IN, OUT: (no value), pinhead:PINHD-1X2
- added 2C1, 2C8: 10m, rcl:CPOL-EUE2.5-5
- added 2C3: 100m, rcl:CPOL-EUE2.5-6
- added 2C4*: 330, rcl:C-EU050-025X075
- added 2C5: 470, rcl:C-EU050-030X075
- added 2C6: 100n, rcl:C-EU075-052X106
- added 2C7: 100m, rcl:CPOL-EUE2.5-5
- added 2C9: 2000m(10000m), rcl:CPOL-EUE5-13
- added 2R1: 15k, rcl:R-EU_R0805
- added 2R10*: 1k, rcl:R-EU_0207/12
- added 2R2: 150k, rcl:R-EU_R0805
- added 2R3: 47k, rcl:R-TRIMM3296W
- added 2R4, 2R5: 10k, rcl:R-EU_R0805
- added 2R6: 330, rcl:R-EU_R0805
- added 2R7: 5k1, rcl:R-EU_R0805
- added 2R8: 100 0.5w, rcl:R-EU_R1210W
- added 2R8': (no value), rcl:R-EU_R1210W
- added 2R9: 1 0.5w, rcl:R-EU_0411/3V
- added IN2, OUT2: (no value), pinhead:PINHD-1X2
- +12V: device DSS:CON_2P -> untitled:CON_2P
Connections:
- removed net N$27: 1C4.+, IN1.1
- removed net N$7: 1C1.+, IN.1
- new net IN1: 1C1.+, IN1.1
- new net IN2: 2C1.+, IN2.1
- net +12V: now also 2R7.2, 2R8.2; no longer 1R15.2, 1R16.2, C10.+
- net GND: now also 2C3.-, 2C4*.2, 2C9.-, 2R3.E, 2R3.S, 2R6.1, 2R9.2, IN2.2; no longer 1C13.-, 1C18.-, 1C4*1.2, 1R11.1, 1R17.2, 1R18.E, 1R18.S, C10.-, IN.2
- net N$16: now also 2R2.2, 2R5.1; no longer 1R10.1, 1R12.2
- net N$17: now also 2R6.2; no longer 1R11.2
- net N$18: now also 2R1.2, 2R2.1, 2R3.A; no longer 1R12.1, 1R13.2, 1R18.A
- net N$19: now also 2C1.-, 2R1.1; no longer 1C4.-, 1R13.1
- net N$20: now also 2C8.+, 2R4.1, 2R5.2; no longer 1C17.+, 1R10.2, 1R14.1
- net N$21: now also 2R4.2, 2R7.1; no longer 1R14.2, 1R15.1
- net N$22: now also 2C3.+; no longer 1C13.+
- net N$23: now also 2C7.+, 2R8'.1; no longer 1C14.+, 1R8'1.1
- net N$24: now also 2C4*.1, 2C5.2; no longer 1C15.2, 1C4*1.1
- net N$25: now also 2C6.2, 2R9.1; no longer 1C16.2, 1R17.1
- net N$26: now also 2C8.-, 2R10*.1; no longer 1C17.-, 1R10*1.1
- net N$28: now also 2R8'.2, 2R8.1; no longer 1R16.1, 1R8'1.2
- net OUT1+: now also OUT1.1; no longer OUT.1
- net OUT1-: now also OUT1.2; no longer OUT.2
- net OUT2+: now also 2C5.1, 2C6.1, 2C7.-, OUT2.1; no longer 1C14.-, 1C15.1, 1C16.1, OUT1.1
- net OUT2-: now also 2C9.+, 2R10*.2, OUT2.2; no longer 1C18.+, 1R10*1.2, OUT1.2
Other:
- note added: "УМЗЧ с малыми искажениями на ИС К174УН7"
- moved on the sheet: +12V, 1C1, 1C10, 1C2, 1C3, 1C4*, 1C5, 1C6, 1C7, 1C8, 1C9, 1R1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
