File: AMP_UN7+T.sch (EAGLE design)
At the start: 54 parts

Commit message: 7
Connections:
- net GND: now also 1R9.1; no longer 1R9.2
- net N$12: now also 1R9.2; no longer 1R9.1
Other:
- moved on the sheet: 1R9
Changed lines of the file:
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@@
 <instance part="1C5" gate="G$1" x="101.6" y="114.3"/>
 <instance part="1C6" gate="G$1" x="109.22" y="114.3"/>
-<instance part="1R9" gate="G$1" x="109.22" y="101.6" smashed="yes" rot="MR270">
-<attribute name="NAME" x="110.49" y="102.6414" size="1.778" layer="95" rot="MR180"/>
-<attribute name="VALUE" x="110.49" y="104.902" size="1.778" layer="96" rot="MR180"/>
+<instance part="1R9" gate="G$1" x="109.22" y="101.6" smashed="yes" rot="R90">
+<attribute name="NAME" x="110.49" y="100.5586" size="1.778" layer="95"/>
+<attribute name="VALUE" x="110.49" y="98.298" size="1.778" layer="96"/>
 </instance>
 <instance part="GND5" gate="1" x="109.22" y="91.44"/>
@@
 </segment>
 <segment>
-<pinref part="1R9" gate="G$1" pin="2"/>
+<pinref part="1R9" gate="G$1" pin="1"/>
 <pinref part="GND5" gate="1" pin="GND"/>
 <wire x1="109.22" y1="96.52" x2="109.22" y2="93.98" width="0.1524" layer="91"/>
@@
 <segment>
 <pinref part="1C6" gate="G$1" pin="2"/>
-<pinref part="1R9" gate="G$1" pin="1"/>
+<pinref part="1R9" gate="G$1" pin="2"/>
 <wire x1="109.22" y1="109.22" x2="109.22" y2="106.68" width="0.1524" layer="91"/>
 </segment>
